Commit message: Add camera hook link

File: spot_description/urdf/spot.urdf.xacro (robot description, xacro)
@@ -13,4 +13,16 @@
         </collision>
     </link>
+    <link name="camera_link">
+        <visual>
+            <geometry>
+                <mesh filename="package://spot_description/meshes/iphone13.dae" />
+            </geometry>
+        </visual>
+    </link>
+    <joint name="camera_body_joint" type="fixed">
+        <origin xyz="-0.223 0 -0.0805" rpy="0 0 0" />
+        <parent link="camera_link" />
+        <child link="body" />
+    </joint>
     <link name="base_link"/>
     <joint name="base_link_joint" type="fixed">

Commit message: feat: create tf linkage

File: spot_description/urdf/spot.urdf.xacro (robot description, xacro)
@@ -13,16 +13,4 @@
         </collision>
     </link>
-    <link name="camera_link">
-        <visual>
-            <geometry>
-                <mesh filename="package://spot_description/meshes/iphone13.dae" />
-            </geometry>
-        </visual>
-    </link>
-    <joint name="camera_body_joint" type="fixed">
-        <origin xyz="-0.223 0 -0.0805" rpy="0 0 0" />
-        <parent link="camera_link" />
-        <child link="body" />
-    </joint>
     <link name="base_link"/>
     <joint name="base_link_joint" type="fixed">
@@ -36,4 +24,22 @@
         <parent link="body" />
         <child link="front_rail" />
+    </joint>
+    <link name="camera">
+        <visual>
+            <geometry>
+                <mesh filename="package://spot_description/meshes/iphone13.dae" />
+            </geometry>
+        </visual>
+    </link>
+    <joint name="camera_joint" type="fixed">
+        <origin xyz="0.2075 0 0.0805" rpy="0 0 0" />
+        <parent link="body" />
+        <child link="camera" />
+    </joint>
+    <link name="origin" />
+    <joint name="origin_joint" type="fixed">
+        <origin xyz="0 0 0" rpy="0 0 0" />
+        <parent link="camera" />
+        <child link="origin" />
     </joint>
     <link name="real_front_rail"/>

Commit message: fix: change origin to float

File: spot_description/urdf/spot.urdf.xacro (robot description, xacro)
@@ -38,5 +38,5 @@
     </joint>
     <link name="origin" />
-    <joint name="origin_joint" type="fixed">
+    <joint name="origin_joint" type="floating">
         <origin xyz="0 0 0" rpy="0 0 0" />
         <parent link="camera" />
